Commit message: Initial ROS 2 robotics workspace

File: src/my_robot_description/urdf/my_robot.urdf (robot description, URDF)
Before this commit: robot my_diff_drive_robot, 6 links, 5 joints
Links:
- link chassis: mass 1.0 -> 3.0
Joints:
- joint left_wheel_joint: limit (none) -> effort=2.5 velocity=10.0
- joint right_wheel_joint: limit (none) -> effort=2.5 velocity=10.0

Commit message: Stabilize cascaded PID path-tracking benchmark

File: src/my_robot_description/urdf/my_robot.urdf (robot description, URDF)
Before this commit: robot my_diff_drive_robot, 6 links, 5 joints
Joints:
- joint left_wheel_joint: limit effort=2.5 velocity=10.0 -> effort=20.0 velocity=10.0
- joint right_wheel_joint: limit effort=2.5 velocity=10.0 -> effort=20.0 velocity=10.0

Commit message: Add LTV controllers and pre-campaign benchmark suite

File: src/my_robot_description/urdf/my_robot.urdf (robot description, URDF)
Before this commit: robot my_diff_drive_robot, 6 links, 5 joints
Joints:
- joint left_wheel_joint: limit effort=20.0 velocity=10.0 -> effort=20.0 velocity=13.0
- joint right_wheel_joint: limit effort=20.0 velocity=10.0 -> effort=20.0 velocity=13.0
